Commit message: modificacion de preuba de git

File: src/modelrobot_pkg_ga/model/robot_car_ga.urdf.xacro (robot description, xacro)
@@ -1,5 +1,5 @@
 <?xml version='1.0'?>
 <robot xmlns:xacro="http://www.ros.org/wiki/xacro" name="robot_car">
-    <xacro:property name="blx" value="${10/10}" />
+    <xacro:property name="blx" value="${10/9}" />
     <xacro:property name="bly" value="${8/10}" />
     <xacro:property name="blz" value="${5/10}" />
